File: mcuModule.sch (EAGLE design)
At the start: 13 parts, among them J1 PRGM, U4 NCP1117ST50T3G, U7 ATMEGA328P

Commit message: added board layout and gerber files
Parts:
- removed JP4: M02PTH, SparkFun-Connectors:M02PTH
- added JP1, JP2: M15, SparkFun-Connectors:M15
- added JP3: (no value), SparkFun-Connectors:M03PTH
Connections:
- net N$1 renamed PB6
- net N$2 renamed PB7
- new net REG_OUT: C7.+, JP3.1, U4.OUT, U4.TAB
- new net VIN_5V: JP1.15, JP3.3
- net 5V: now also JP1.13, JP3.2; no longer C7.+, U4.OUT, U4.TAB
- net ADC0: now also JP2.9
- net ADC1: now also JP2.8
- net ADC2: now also JP2.7
- net ADC3: now also JP2.6
- net ADC6: now also JP2.11
- net ADC7: now also JP2.10
- net AREF: now also JP2.13
- net GND: now also JP1.12, JP2.14, JP2.15; no longer JP4.1
- net MISO: now also JP1.4
- net MOSI: now also JP1.5
- net PB0: now also JP1.8
- net PB1: now also JP1.7
- net PB2: now also JP1.6
- net PD2: now also JP2.1
- net PD3: now also JP1.1
- net PD4: now also JP1.2
- net PD5: now also JP1.11
- net PD6: now also JP1.10
- net PD7: now also JP1.9
- net RESET: now also JP2.12
- net RXD: now also JP2.3
- net SCK: now also JP1.3
- net SCL: now also JP2.4
- net SDA: now also JP2.5
- net TXD: now also JP2.2
- net VIN: now also JP1.14; no longer JP4.2
Other:
- note added: "Status LEDs"
- moved on the sheet: C1, C3, C7, J1, LED4, R1, R10, S1, U4, U7, Y1
